File: power_2019.kicad_pcb (KiCad board)
At the start: 2 copper layers, 0 parts

Commit message: update power board
Parts:
- added D1: LED_12V_rouge, LED_SMD:LED_1206_3216Metric_Pad1.42x1.75mm_HandSolder, F.Cu at (178.6, 96.9)
- added D3: 1N5822, Diode_THT:D_DO-201AD_P15.24mm_Horizontal, F.Cu at (167.4, 78.2)
- added D4: 1N5822, Diode_THT:D_DO-201AD_P15.24mm_Horizontal, F.Cu at (167.4, 85.6)
- added J1: Alim logique, TerminalBlock_Phoenix:TerminalBlock_Phoenix_MPT-0,5-2-2.54_1x02_P2.54mm_Horizontal, F.Cu at (178.1, 92.1)
- added J2: Alim puissance, TerminalBlock_Phoenix:TerminalBlock_Phoenix_MPT-0,5-2-2.54_1x02_P2.54mm_Horizontal, F.Cu at (184.6, 94.6)
- added R1: 1k, Resistor_SMD:R_1206_3216Metric_Pad1.42x1.75mm_HandSolder, F.Cu at (191.7, 92.1)
- added U1: PTH08080W, @Robot_symbols:PTH08080W, F.Cu at (184.7, 77.2)
- added U2: LM2576T-ADJ, Package_TO_SOT_THT:TO-220-5_Vertical, F.Cu at (167.4, 96.8)
- added U3: LM2576T-ADJ, Package_TO_SOT_THT:TO-220-5_Vertical, F.Cu at (167.4, 91.9)
