File: power_7_4V/power_7_4V.kicad_pcb (KiCad board)
At the start: 2 copper layers, 82.5 x 26.7 mm, 13 parts, among them J1 Alim_Batt, J2 Alim_Servo, J3 Conn_Facade, U1 LM2576T-ADJ

Commit message: maj servo
Routing:
- net /7,4V_OUT: track 0.00 -> 15.2 mm
- net Net-(D2-Pad2): track 0.00 -> 3.81 mm
- added copper zone on B.Cu, net (none)
Other:
- board text added: "Club Robot 2019 Carte Alim Servo - Boyer Norman"
Changed lines of the file:
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@@
   (general
     (thickness 1.6)
-    (drawings 4)
-    (tracks 31)
+    (drawings 5)
+    (tracks 37)
     (zones 0)
     (modules 13)
@@
     (solder_mask_min_width 0.25)
     (aux_axis_origin 0 0)
-    (visible_elements FFFFF77F)
+    (visible_elements FFFFFF7F)
     (pcbplotparams
       (layerselection 0x010fc_ffffffff)
@@
     )
   )
+  (gr_text "Club Robot 2019\nCarte Alim Servo - Boyer Norman" (at 100.33 88.9) (layer B.Cu)
+    (effects (font (size 1 1) (thickness 0.25)) (justify mirror))
+  )
   (gr_line (start 162.56 67.31) (end 80.01 67.31) (layer Edge.Cuts) (width 0.15))
   (gr_line (start 162.56 93.98) (end 162.56 67.31) (layer Edge.Cuts) (width 0.15))
@@
   (segment (start 136.93 72.16) (end 137.16 72.39) (width 0.762) (layer B.Cu) (net 4))
   (segment (start 124.46 72.16) (end 136.93 72.16) (width 0.762) (layer B.Cu) (net 4))
+  (segment (start 158.75 80.01) (end 158.75 83.82) (width 0.762) (layer B.Cu) (net 5))
   (segment (start 97.7 76.2) (end 97.77 76.27) (width 0.762) (layer B.Cu) (net 6))
   (segment (start 91.44 76.2) (end 97.7 76.2) (width 0.762) (layer B.Cu) (net 6))
+  (segment (start 146.05 72.916253) (end 146.05 74.93) (width 0.762) (layer B.Cu) (net 8))
+  (segment (start 146.05 74.93) (end 147.32 76.2) (width 0.762) (layer B.Cu) (net 8))
+  (segment (start 147.32 76.2) (end 154.94 76.2) (width 0.762) (layer B.Cu) (net 8))
+  (segment (start 154.94 76.2) (end 156.21 74.93) (width 0.762) (layer B.Cu) (net 8))
+  (segment (start 156.21 74.93) (end 156.21 72.916253) (width 0.762) (layer B.Cu) (net 8))
   (segment (start 128.27 91.44) (end 130.81 88.9) (width 0.762) (layer B.Cu) (net 11))
   (segment (start 121.92 91.44) (end 128.27 91.44) (width 0.762) (layer B.Cu) (net 11))
@@
   (segment (start 119.38 88.9) (end 121.92 91.44) (width 0.762) (layer B.Cu) (net 11))
   (segment (start 143.51 80.01) (end 143.51 83.82) (width 0.762) (layer B.Cu) (net 11))
+  (zone (net 0) (net_name "") (layer B.Cu) (hatch edge 0.508)
+    (connect_pads (clearance 0.508))
+    (min_thickness 0.254)
+    (fill yes (arc_segments 16) (thermal_gap 0.508) (thermal_bridge_width 0.508))
+    (polygon
+      (pts
+        (xy 81.28 68.58) (xy 81.28 92.71) (xy 161.29 92.71) (xy 161.29 68.58)
+      )
+    )
+  )
 )
